Commit message: fix leap left problem

File: leap_description/robots/leap_left.urdf (robot description, URDF)
Before this commit: robot onshape, 17 links, 16 joints
Links:
- removed link palm_lower_left
- added link palm_lower, mass 0.235; collision mesh filename=package://leap_description/meshes/palm_lower_left.stl; visual mesh filename=package://leap_description/meshes/palm_lower_left.stl
Joints:
- joint joint_1: parent palm_lower_left -> palm_lower
- joint joint_12: child thumb_pip -> thumb_left_temp_base; limit lower=-2.094 upper=0.349 effort=0.95 velocity=8.48 -> lower=-2.443 upper=0.47 effort=0.95 velocity=8.48; origin xyz=-1.0148132334464321502e-16 -0.014100000000000126321 -0.012999999999999956035 rpy=-1.570796326794896336 -1.570796326794896336 0 -> xyz=-0.14487422493839263726 -0.090040011501137440231 0.004900888583899039308 rpy=3.5629789726327258012e-15 1.5707963267948961139 0; parent thumb_left_temp_base -> palm_lower
- joint joint_13: child thumb_left_temp_base -> thumb_pip; limit lower=-2.443 upper=0.47 effort=0.95 velocity=8.48 -> lower=-2.094 upper=0.349 effort=0.95 velocity=8.48; origin xyz=-0.14487422493839263726 -0.090040011501137440231 0.004900888583899039308 rpy=3.5629789726327258012e-15 1.5707963267948961139 0 -> xyz=-1.0148132334464321502e-16 -0.014100000000000126321 -0.012999999999999956035 rpy=-1.570796326794896336 -1.570796326794896336 0; parent palm_lower_left -> thumb_left_temp_base
- joint joint_5: parent palm_lower_left -> palm_lower
- joint joint_9: parent palm_lower_left -> palm_lower
